Commit message: Rename: base_0 -> base_link, extended m1013
m1013 (white): param "prefix", additional links base, flange and tool0

File: dsr_description/config/macro.gazebo.xacro (robot description, xacro)
@@ -7,5 +7,5 @@
             <selfCollide>true</selfCollide>
         </gazebo>
-		<gazebo reference="base_0">
+		<gazebo reference="base_link">
             <selfCollide>true</selfCollide>
 			<kp>1000000.0</kp>

File: dsr_description/urdf/m0609.urdf (robot description, URDF)
Before this commit: robot m0609, 8 links, 7 joints
Links:
- removed link base_0
- added link base_link, mass 3.722; visual mesh filename=package://dsr_description/meshes/m0609/MF0609_0_0.dae scale=0.001 0.001 0.001
Joints:
- joint fixed: child base_0 -> base_link
- joint joint1: parent base_0 -> base_link

File: dsr_description/urdf/m0617.urdf (robot description, URDF)
Before this commit: robot m0617, 8 links, 7 joints
Links:
- removed link base_0
- added link base_link, mass 3.722; visual mesh filename=package://dsr_description/meshes/m0617/MF0617_0_0.dae scale=0.001 0.001 0.001
Joints:
- joint fixed: child base_0 -> base_link
- joint joint1: parent base_0 -> base_link

File: dsr_description/urdf/m1013.urdf (robot description, URDF)
Before this commit: robot m1013, 8 links, 7 joints
Links:
- removed link base_0
- added link base_link, mass 3.722; visual mesh filename=package://dsr_description/meshes/m1013/MF1013_0_0.dae scale=0.001 0.001 0.001
Joints:
- joint fixed: child base_0 -> base_link
- joint joint1: parent base_0 -> base_link

File: dsr_description/urdf/m1509.urdf (robot description, URDF)
Before this commit: robot m1509, 8 links, 7 joints
Links:
- removed link base_0
- added link base_link, mass 3.722; visual mesh filename=package://dsr_description/meshes/m1509/MF1509_0_0.dae scale=0.001 0.001 0.001
Joints:
- joint fixed: child base_0 -> base_link
- joint joint1: parent base_0 -> base_link

File: dsr_description/xacro/a0509.urdf.xacro (robot description, xacro)
@@ -20,5 +20,5 @@
     <origin xyz="0 0 0" rpy="0 0 0"/>
     <parent link="world"/>
-    <child link="base_0"/>
+    <child link="base_link"/>
   </joint>
 </robot>

File: dsr_description/xacro/m0609.urdf.xacro (robot description, xacro)
@@ -20,5 +20,5 @@
     <origin xyz="0 0 0" rpy="0 0 0"/>
     <parent link="world"/>
-    <child link="base_0"/>
+    <child link="base_link"/>
   </joint>
 </robot>

File: dsr_description/xacro/m0617.urdf.xacro (robot description, xacro)
@@ -20,5 +20,5 @@
     <origin xyz="0 0 0" rpy="0 0 0"/>
     <parent link="world"/>
-    <child link="base_0"/>
+    <child link="base_link"/>
   </joint>
 </robot>

File: dsr_description/xacro/m1013.urdf.xacro (robot description, xacro)
@@ -20,5 +20,5 @@
     <origin xyz="0 0 0" rpy="0 0 0"/>
     <parent link="world"/>
-    <child link="base_0"/>
+    <child link="base_link"/>
   </joint>
 </robot>

File: dsr_description/xacro/m1509.urdf.xacro (robot description, xacro)
@@ -20,5 +20,5 @@
     <origin xyz="0 0 0" rpy="0 0 0"/>
     <parent link="world"/>
-    <child link="base_0"/>
+    <child link="base_link"/>
   </joint>
 </robot>

File: dsr_description/xacro/macro.a0509.blue.xacro (robot description, xacro)
@@ -6,5 +6,5 @@
 	<xacro:macro name="a0509" params="namespace">
 		<xacro:dsr_materials />
-		<link name="base_0">
+		<link name="base_link">
 			<inertial>
 				<mass value="2.198"/>
@@ -23,5 +23,5 @@
 		<!-- joint 1 -->
 		<joint name="joint1" type="revolute">
-			<parent link="base_0" />
+			<parent link="base_link" />
 			<child link="link1" />
 			<origin rpy="0 0 0" xyz="0 0 0.1555" />

File: dsr_description/xacro/macro.a0509mobile.blue.xacro (robot description, xacro)
@@ -85,5 +85,5 @@
 		<joint name="dsr_arm_base" type="fixed">
 			<parent link="top_plate_link" />
-			<child link="base_0" />
+			<child link="base_link" />
 			<origin xyz="0 0 0.0065" rpy="0.0 0.0 -1.57" />
 		</joint>

File: dsr_description/xacro/macro.m0609.blue.xacro (robot description, xacro)
@@ -6,5 +6,5 @@
 	<xacro:macro name="m0609" params="namespace">
     <xacro:dsr_materials />
-		<link name="base_0">
+		<link name="base_link">
 			<inertial>
 				<mass value="3.18"/>
@@ -23,5 +23,5 @@
 		<!-- joint 1 -->
 		<joint name="joint1" type="revolute">
-			<parent link="base_0" />
+			<parent link="base_link" />
 			<child link="link1" />
 			<origin rpy="0 0 0" xyz="0 0 0.1" />

File: dsr_description/xacro/macro.m0609.white.xacro (robot description, xacro)
@@ -6,5 +6,5 @@
 	<xacro:macro name="m0609" params="namespace">
     <xacro:dsr_materials />
-		<link name="base_0">
+		<link name="base_link">
 			<inertial>
 				<mass value="3.18"/>
@@ -23,5 +23,5 @@
 		<!-- joint 1 -->
 		<joint name="joint1" type="revolute">
-			<parent link="base_0" />
+			<parent link="base_link" />
 			<child link="link1" />
 			<origin rpy="0 0 0" xyz="0 0 0.1" />

File: dsr_description/xacro/macro.m0609mobile.blue.xacro (robot description, xacro)
@@ -87,5 +87,5 @@
 		<joint name="dsr_arm_base" type="fixed">
 			<parent link="top_plate_link" />
-			<child link="base_0" />
+			<child link="base_link" />
 			<origin xyz="0 0 0.0065" rpy="0.0 0.0 -1.57" />
 		</joint>

File: dsr_description/xacro/macro.m0609mobile.white.xacro (robot description, xacro)
@@ -87,5 +87,5 @@
 		<joint name="dsr_arm_base" type="fixed">
 			<parent link="top_plate_link" />
-			<child link="base_0" />
+			<child link="base_link" />
 			<origin xyz="0 0 0.0065" rpy="0.0 0.0 -1.57" />
 		</joint>

File: dsr_description/xacro/macro.m0617.blue.xacro (robot description, xacro)
@@ -6,5 +6,5 @@
 	<xacro:macro name="m0617" params="namespace">
 		<xacro:dsr_materials />
-		<link name="base_0">
+		<link name="base_link">
 			<inertial>
 				<mass value="4.12"/>
@@ -23,5 +23,5 @@
 		<!-- joint 1 -->
 		<joint name="joint1" type="revolute">
-			<parent link="base_0" />
+			<parent link="base_link" />
 			<child link="link1" />
 			<origin rpy="0 0 0" xyz="0 0 0.1525" />

File: dsr_description/xacro/macro.m0617.white.xacro (robot description, xacro)
@@ -6,5 +6,5 @@
 	<xacro:macro name="m0617" params="namespace">
 		<xacro:dsr_materials />
-		<link name="base_0">
+		<link name="base_link">
 			<inertial>
 				<mass value="4.12"/>
@@ -23,5 +23,5 @@
 		<!-- joint 1 -->
 		<joint name="joint1" type="revolute">
-			<parent link="base_0" />
+			<parent link="base_link" />
 			<child link="link1" />
 			<origin rpy="0 0 0" xyz="0 0 0.1525" />

File: dsr_description/xacro/macro.m0617mobile.blue.xacro (robot description, xacro)
@@ -85,5 +85,5 @@
 		<joint name="dsr_arm_base" type="fixed">
 			<parent link="top_plate_link" />
-			<child link="base_0" />
+			<child link="base_link" />
 			<origin xyz="0 0 0.0065" rpy="0.0 0.0 -1.57" />
 		</joint>

File: dsr_description/xacro/macro.m0617mobile.white.xacro (robot description, xacro)
@@ -85,5 +85,5 @@
 		<joint name="dsr_arm_base" type="fixed">
 			<parent link="top_plate_link" />
-			<child link="base_0" />
+			<child link="base_link" />
 			<origin xyz="0 0 0.0065" rpy="0.0 0.0 -1.57" />
 		</joint>
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