Commit message: Rename: base_0 -> base_link, extended m1013
m1013 (white): param "prefix", additional links base, flange and tool0

File: dsr_description/xacro/macro.m1013.white.xacro (robot description, xacro)
@@ -4,7 +4,7 @@
   <xacro:include filename="$(find dsr_description)/config/macro.transmission.xacro"/>
   <xacro:include filename="$(find dsr_description)/config/macro.materials.xacro"/>
-  <xacro:macro name="m1013" params="namespace">
+  <xacro:macro name="m1013" params="prefix:='' namespace:=''">
     <xacro:dsr_materials/>
-    <link name="base_0">
+    <link name="${prefix}base_link">
       <inertial>
         <mass value="4.12"/>
@@ -25,7 +25,7 @@
     </link>
     <!-- joint 1 -->
-    <joint name="joint1" type="revolute">
-      <parent link="base_0"/>
-      <child link="link1"/>
+    <joint name="${prefix}joint1" type="revolute">
+      <parent link="${prefix}base_link"/>
+      <child link="${prefix}link1"/>
       <origin rpy="0 0 0" xyz="0 0 0.1525"/>
       <axis xyz="0 0 1"/>
@@ -33,5 +33,5 @@
       <dynamics friction="0"/>
     </joint>
-    <link name="link1">
+    <link name="${prefix}link1">
       <inertial>
         <mass value="7.8"/>
@@ -52,7 +52,7 @@
     </link>
     <!-- joint2 -->
-    <joint name="joint2" type="revolute">
-      <parent link="link1"/>
-      <child link="link2"/>
+    <joint name="${prefix}joint2" type="revolute">
+      <parent link="${prefix}link1"/>
+      <child link="${prefix}link2"/>
       <origin rpy="0 -${pi/2} -${pi/2}" xyz="0 0.0345 0"/>
       <axis xyz="0 0 1"/>
@@ -60,5 +60,5 @@
       <dynamics friction="0"/>
     </joint>
-    <link name="link2">
+    <link name="${prefix}link2">
       <inertial>
         <mass value="10.83"/>
@@ -99,7 +99,7 @@
     </link>
     <!-- joint3 -->
-    <joint name="joint3" type="revolute">
-      <parent link="link2"/>
-      <child link="link3"/>
+    <joint name="${prefix}joint3" type="revolute">
+      <parent link="${prefix}link2"/>
+      <child link="${prefix}link3"/>
       <origin rpy="0 0 ${pi/2}" xyz="0.62 0 0"/>
       <axis xyz="0 0 1"/>
@@ -107,5 +107,5 @@
       <dynamics friction="0"/>
     </joint>
-    <link name="link3">
+    <link name="${prefix}link3">
       <inertial>
         <mass value="3.68"/>
@@ -126,7 +126,7 @@
     </link>
     <!-- joint4 -->
-    <joint name="joint4" type="revolute">
-      <parent link="link3"/>
-      <child link="link4"/>
+    <joint name="${prefix}joint4" type="revolute">
+      <parent link="${prefix}link3"/>
+      <child link="${prefix}link4"/>
       <origin rpy="${pi/2} 0 0" xyz="0 -0.559 0"/>
       <axis xyz="0 0 1"/>
@@ -134,5 +134,5 @@
       <dynamics friction="0"/>
     </joint>
-    <link name="link4">
+    <link name="${prefix}link4">
       <inertial>
         <mass value="3.82"/>
@@ -163,7 +163,7 @@
     </link>
     <!-- joint5 -->
-    <joint name="joint5" type="revolute">
-      <parent link="link4"/>
-      <child link="link5"/>
+    <joint name="${prefix}joint5" type="revolute">
+      <parent link="${prefix}link4"/>
+      <child link="${prefix}link5"/>
       <origin rpy="-${pi/2} 0 0" xyz="0 0 0"/>
       <axis xyz="0 0 1"/>
@@ -171,5 +171,5 @@
       <dynamics friction="0"/>
     </joint>
-    <link name="link5">
+    <link name="${prefix}link5">
       <inertial>
         <mass value="2.82"/>
@@ -190,7 +190,7 @@
     </link>
     <!-- joint6 -->
-    <joint name="joint6" type="revolute">
-      <parent link="link5"/>
-      <child link="link6"/>
+    <joint name="${prefix}joint6" type="revolute">
+      <parent link="${prefix}link5"/>
+      <child link="${prefix}link6"/>
       <origin rpy="${pi/2} 0 0" xyz="0 -0.121 0"/>
       <axis xyz="0 0 1"/>
@@ -198,5 +198,5 @@
       <dynamics friction="0"/>
     </joint>
-    <link name="link6">
+    <link name="${prefix}link6">
       <inertial>
         <mass value="1.16"/>
@@ -216,4 +216,25 @@
       </collision>
     </link>
+    <!-- TODO ROS base_link to Doosan Coordinates transform -->
+    <link name="${prefix}base"/>
+    <joint name="${prefix}base_link-base" type="fixed">
+      <origin xyz="0 0 0" rpy="0 0 0"/>
+      <parent link="${prefix}base_link"/>
+      <child link="${prefix}base"/>
+    </joint>
+    <!-- TODO ROS-Industrial 'flange' frame: attachment point for EEF models -->
+    <link name="${prefix}flange"/>
+    <joint name="${prefix}joint6-flange" type="fixed">
+      <origin xyz="0 0 0" rpy="0 0 0"/>
+      <parent link="${prefix}link6"/>
+      <child link="${prefix}flange"/>
+    </joint>
+    <!-- TODO ROS-Industrial 'tool0' frame: all-zeros tool frame -->
+    <link name="${prefix}tool0"/>
+    <joint name="${prefix}link6-tool0" type="fixed">
+      <origin xyz="0 0 0" rpy="0 0 0"/>
+      <parent link="${prefix}flange"/>
+      <child link="${prefix}tool0"/>
+    </joint>
     <xacro:dsr_transmission/>
     <xacro:dsr_gazebo namespace="${namespace}"/>

File: dsr_description/xacro/macro.m1509.blue.xacro (robot description, xacro)
@@ -6,5 +6,5 @@
 	<xacro:macro name="m1509" params="namespace">
 		<xacro:dsr_materials />
-		<link name="base_0">
+		<link name="base_link">
 			<inertial>
 				<mass value="4.12"/>
@@ -23,5 +23,5 @@
 		<!-- joint 1 -->
 		<joint name="joint1" type="revolute">
-			<parent link="base_0" />
+			<parent link="base_link" />
 			<child link="link1" />
 			<origin rpy="0 0 0" xyz="0 0 0.1525" />

Commit message: Made whitespaces/tab indent consistent

File: dsr_description/xacro/macro.m1013.white.xacro (robot description, xacro)
@@ -1,70 +1,70 @@
 <?xml version="1.0"?>
 <robot name="m1013" xmlns:xacro="http://www.ros.org/wiki/xacro">
-	<xacro:include filename="$(find dsr_description)/config/macro.gazebo.xacro" />
-	<xacro:include filename="$(find dsr_description)/config/macro.transmission.xacro" />
-	<xacro:include filename="$(find dsr_description)/config/macro.materials.xacro" />
-	<xacro:macro name="m1013" params="namespace">
-		<xacro:dsr_materials />
-		<link name="base_0">
-			<inertial>
-				<mass value="4.12"/>
-				<origin xyz="-3.4e-05   -0.004815    0.048482"/>
-				<inertia ixx="0.016331" ixy="-6.4837e-06" ixz="2.0048e-06" iyy="0.014945"
-					iyz="-0.00051686"
-					izz="0.022577"/>
-			</inertial>
-			<visual>
-				<origin rpy="0 0 0" xyz="0 0 0" />
-				<geometry>
-					<mesh filename="package://dsr_description/meshes/m1013_white/MF1013_0_0.dae" scale="0.001 0.001 0.001" />
-				</geometry>
-			</visual>
-		</link>
-		<!-- joint 1 -->
-		<joint name="joint1" type="revolute">
-			<parent link="base_0" />
-			<child link="link1" />
-			<origin rpy="0 0 0" xyz="0 0 0.1525" />
-			<axis xyz="0 0 1" />
-			<limit effort="346" lower="-6.2832" upper="6.2832" velocity="2.0944"/>
-			<dynamics friction="0" />
-		</joint>
-		<link name="link1">
-			<inertial>
-				<mass value="7.8"/>
-				<origin xyz="0.000119      0.0428   -0.006383"/>
-				<inertia ixx="0.04506" ixy="4.1126e-05" ixz="-5.2533e-05" iyy="0.029679"
-					iyz="-0.0019959"
-					izz="0.047056"/>
-			</inertial>
-            <collision>
-                <geometry>
-                    <cylinder radius="0.1" length="0.2"/>
-                </geometry>
-            </collision>
-			<visual>
-				<origin rpy="0 0 0" xyz="0 0 0" />
-				<geometry>
-					<mesh filename="package://dsr_description/meshes/m1013_white/MF1013_1_0.dae" scale="0.001 0.001 0.001" />
-				</geometry>
-			</visual>
-		</link>
-		<!-- joint2 -->
-		<joint name="joint2" type="revolute">
-			<parent link="link1" />
-			<child link="link2" />
-			<origin rpy="0 -1.571 -1.571" xyz="0 0.0345 0" />
-			<axis xyz="0 0 1" />
-			<limit effort="346" lower="-6.2832" upper="6.2832" velocity="2.0944"/>
-			<dynamics friction="0" />
-		</joint>
-		<link name="link2">
-			<inertial>
-				<mass value="10.83"/>
-				<origin xyz="0.25973    -5.3e-05     0.15782"/>
-				<inertia ixx="0.037586" ixy="-0.00036999" ixz="-0.0069927" iyy="0.84943"
-					iyz="4.0201e-05"
-					izz="0.85021"/>
-			</inertial>
+  <xacro:include filename="$(find dsr_description)/config/macro.gazebo.xacro" />
+  <xacro:include filename="$(find dsr_description)/config/macro.transmission.xacro" />
+  <xacro:include filename="$(find dsr_description)/config/macro.materials.xacro" />
+  <xacro:macro name="m1013" params="namespace">
+    <xacro:dsr_materials />
+    <link name="base_0">
+      <inertial>
+        <mass value="4.12"/>
+        <origin xyz="-3.4e-05   -0.004815    0.048482"/>
+        <inertia ixx="0.016331" ixy="-6.4837e-06" ixz="2.0048e-06" iyy="0.014945"
+          iyz="-0.00051686"
+          izz="0.022577"/>
+      </inertial>
+      <visual>
+        <origin rpy="0 0 0" xyz="0 0 0" />
+        <geometry>
+          <mesh filename="package://dsr_description/meshes/m1013_white/MF1013_0_0.dae" scale="0.001 0.001 0.001" />
+        </geometry>
+      </visual>
+    </link>
+    <!-- joint 1 -->
+    <joint name="joint1" type="revolute">
+      <parent link="base_0" />
+      <child link="link1" />
+      <origin rpy="0 0 0" xyz="0 0 0.1525" />
+      <axis xyz="0 0 1" />
+      <limit effort="346" lower="-6.2832" upper="6.2832" velocity="2.0944"/>
+      <dynamics friction="0" />
+    </joint>
+    <link name="link1">
+      <inertial>
+        <mass value="7.8"/>
+        <origin xyz="0.000119      0.0428   -0.006383"/>
+        <inertia ixx="0.04506" ixy="4.1126e-05" ixz="-5.2533e-05" iyy="0.029679"
+          iyz="-0.0019959"
+          izz="0.047056"/>
+      </inertial>
+      <collision>
+        <geometry>
+          <cylinder radius="0.1" length="0.2"/>
+        </geometry>
+      </collision>
+      <visual>
+        <origin rpy="0 0 0" xyz="0 0 0" />
+        <geometry>
+          <mesh filename="package://dsr_description/meshes/m1013_white/MF1013_1_0.dae" scale="0.001 0.001 0.001" />
+        </geometry>
+      </visual>
+    </link>
+    <!-- joint2 -->
+    <joint name="joint2" type="revolute">
+      <parent link="link1" />
+      <child link="link2" />
+      <origin rpy="0 -1.571 -1.571" xyz="0 0.0345 0" />
+      <axis xyz="0 0 1" />
+      <limit effort="346" lower="-6.2832" upper="6.2832" velocity="2.0944"/>
+      <dynamics friction="0" />
+    </joint>
+    <link name="link2">
+      <inertial>
+        <mass value="10.83"/>
+        <origin xyz="0.25973    -5.3e-05     0.15782"/>
+        <inertia ixx="0.037586" ixy="-0.00036999" ixz="-0.0069927" iyy="0.84943"
+          iyz="4.0201e-05"
+          izz="0.85021"/>
+      </inertial>
             <collision>
                 <origin rpy="0 -1.571 0" xyz="0.3 0 0.1525" />
@@ -73,63 +73,63 @@
                 </geometry>
             </collision>
-			<visual>
-				<origin rpy="0 0 0" xyz="0 0 0" />
-				<geometry>
-					<mesh filename="package://dsr_description/meshes/m1013_white/MF1013_2_0.dae" scale="0.001 0.001 0.001" />
-				</geometry>
-			</visual>
-			<visual>
-				<origin rpy="0 0 0" xyz="0 0 0" />
-				<geometry>
-					<mesh filename="package://dsr_description/meshes/m1013_white/MF1013_2_1.dae" scale="0.001 0.001 0.001" />
-				</geometry>
-			</visual>
-			<visual>
-				<origin rpy="0 0 0" xyz="0 0 0" />
-				<geometry>
-					<mesh filename="package://dsr_description/meshes/m1013_white/MF1013_2_2.dae" scale="0.001 0.001 0.001" />
-				</geometry>
-			</visual>
-		</link>
-		<!-- joint3 -->
-		<joint name="joint3" type="revolute">
-			<parent link="link2" />
-			<child link="link3" />
-			<origin rpy="0 0 1.571" xyz="0.62 0 0" />
-			<axis xyz="0 0 1" />
-			<limit effort="163" lower="-2.7925" upper="2.7925" velocity="3.1416"/>
-			<dynamics friction="0" />
-		</joint>
-		<link name="link3">
-			<inertial>
-				<mass value="3.68"/>
-				<origin xyz="-1.5e-05   -0.006702    0.044608"/>
-				<inertia ixx="0.018748" ixy="7.8071e-06" ixz="-5.0324e-06" iyy="0.018972"
-					iyz="-0.00099342"
-					izz="0.011502"/>
-			</inertial>
+      <visual>
+        <origin rpy="0 0 0" xyz="0 0 0" />
+        <geometry>
+          <mesh filename="package://dsr_description/meshes/m1013_white/MF1013_2_0.dae" scale="0.001 0.001 0.001" />
+        </geometry>
+      </visual>
+      <visual>
+        <origin rpy="0 0 0" xyz="0 0 0" />
+        <geometry>
+          <mesh filename="package://dsr_description/meshes/m1013_white/MF1013_2_1.dae" scale="0.001 0.001 0.001" />
+        </geometry>
+      </visual>
+      <visual>
+        <origin rpy="0 0 0" xyz="0 0 0" />
+        <geometry>
+          <mesh filename="package://dsr_description/meshes/m1013_white/MF1013_2_2.dae" scale="0.001 0.001 0.001" />
+        </geometry>
+      </visual>
+    </link>
+    <!-- joint3 -->
+    <joint name="joint3" type="revolute">
+      <parent link="link2" />
+      <child link="link3" />
+      <origin rpy="0 0 1.571" xyz="0.62 0 0" />
+      <axis xyz="0 0 1" />
+      <limit effort="163" lower="-2.7925" upper="2.7925" velocity="3.1416"/>
+      <dynamics friction="0" />
+    </joint>
+    <link name="link3">
+      <inertial>
+        <mass value="3.68"/>
+        <origin xyz="-1.5e-05   -0.006702    0.044608"/>
+        <inertia ixx="0.018748" ixy="7.8071e-06" ixz="-5.0324e-06" iyy="0.018972"
+          iyz="-0.00099342"
+          izz="0.011502"/>
+      </inertial>
             <visual>
-				<origin rpy="0 0 0" xyz="0 0 0" />
-				<geometry>
-					<mesh filename="package://dsr_description/meshes/m1013_white/MF1013_3_0.dae" scale="0.001 0.001 0.001" />
-				</geometry>
-			</visual>
-		</link>
-		<!-- joint4 -->
-		<joint name="joint4" type="revolute">
-			<parent link="link3" />
-			<child link="link4" />
-			<origin rpy="1.571 0 0" xyz="0 -0.559 0" />
-			<axis xyz="0 0 1" />
-			<limit effort="50" lower="-6.2832" upper="6.2832" velocity="3.927"/>
-			<dynamics friction="0" />
-		</joint>
-		<link name="link4">
-			<inertial>
-				<mass value="3.82"/>
-				<origin xyz="7.1e-05    0.091879    -0.18252"/>
-				<inertia ixx="0.19063" ixy="-1.8037e-05" ixz="-3.8576e-05" iyy="0.17268" iyz="-0.052996"
-					izz="0.030386"/>
-			</inertial>
+        <origin rpy="0 0 0" xyz="0 0 0" />
+        <geometry>
+          <mesh filename="package://dsr_description/meshes/m1013_white/MF1013_3_0.dae" scale="0.001 0.001 0.001" />
+        </geometry>
+      </visual>
+    </link>
+    <!-- joint4 -->
+    <joint name="joint4" type="revolute">
+      <parent link="link3" />
+      <child link="link4" />
+      <origin rpy="1.571 0 0" xyz="0 -0.559 0" />
+      <axis xyz="0 0 1" />
+      <limit effort="50" lower="-6.2832" upper="6.2832" velocity="3.927"/>
+      <dynamics friction="0" />
+    </joint>
+    <link name="link4">
+      <inertial>
+        <mass value="3.82"/>
+        <origin xyz="7.1e-05    0.091879    -0.18252"/>
+        <inertia ixx="0.19063" ixy="-1.8037e-05" ixz="-3.8576e-05" iyy="0.17268" iyz="-0.052996"
+          izz="0.030386"/>
+      </inertial>
             <collision>
                 <origin rpy="-0.55 0 0" xyz="0 0.07 -0.3" />
@@ -138,34 +138,34 @@
                 </geometry>
             </collision>
-			<visual>
-				<origin rpy="0 0 0" xyz="0 0 0" />
-				<geometry>
-					<mesh filename="package://dsr_description/meshes/m1013_white/MF1013_4_0.dae" scale="0.001 0.001 0.001" />
-				</geometry>
-			</visual>
-			<visual>
-				<origin rpy="0 0 0" xyz="0 0 0" />
-				<geometry>
-					<mesh filename="package://dsr_description/meshes/m1013_white/MF1013_4_1.dae" scale="0.001 0.001 0.001" />
-				</geometry>
-			</visual>
-		</link>
-		<!-- joint5 -->
-		<joint name="joint5" type="revolute">
-			<parent link="link4" />
-			<child link="link5" />
-			<origin rpy="-1.571 0 0" xyz="0 0 0" />
-			<axis xyz="0 0 1" />
-			<limit effort="50" lower="-6.2832" upper="6.2832" velocity="3.927"/>
-			<dynamics friction="0" />
-		</joint>
-		<link name="link5">
-			<inertial>
-				<mass value="2.82"/>
-				<origin xyz="-0.000273    0.003651    0.032088"/>
-				<inertia ixx="0.015583" ixy="2.135e-05" ixz="-5.1895e-06" iyy="0.011519"
-					iyz="0.00042553"
-					izz="0.0088671"/>
-			</inertial>
+      <visual>
+        <origin rpy="0 0 0" xyz="0 0 0" />
+        <geometry>
+          <mesh filename="package://dsr_description/meshes/m1013_white/MF1013_4_0.dae" scale="0.001 0.001 0.001" />
+        </geometry>
+      </visual>
+      <visual>
+        <origin rpy="0 0 0" xyz="0 0 0" />
+        <geometry>
+          <mesh filename="package://dsr_description/meshes/m1013_white/MF1013_4_1.dae" scale="0.001 0.001 0.001" />
+        </geometry>
+      </visual>
+    </link>
+    <!-- joint5 -->
+    <joint name="joint5" type="revolute">
+      <parent link="link4" />
+      <child link="link5" />
+      <origin rpy="-1.571 0 0" xyz="0 0 0" />
+      <axis xyz="0 0 1" />
+      <limit effort="50" lower="-6.2832" upper="6.2832" velocity="3.927"/>
+      <dynamics friction="0" />
+    </joint>
+    <link name="link5">
+      <inertial>
+        <mass value="2.82"/>
+        <origin xyz="-0.000273    0.003651    0.032088"/>
+        <inertia ixx="0.015583" ixy="2.135e-05" ixz="-5.1895e-06" iyy="0.011519"
+          iyz="0.00042553"
+          izz="0.0088671"/>
+      </inertial>
             <collision>
                 <origin rpy="1.571 0 0" xyz="0 0 0" />
@@ -174,37 +174,37 @@
                 </geometry>
             </collision>
-			<visual>
-				<origin rpy="0 0 0" xyz="0 0 0" />
-				<geometry>
-					<mesh filename="package://dsr_description/meshes/m1013_white/MF1013_5_0.dae" scale="0.001 0.001 0.001" />
-				</geometry>
-			</visual>
-		</link>
-		<!-- joint6 -->
-		<joint name="joint6" type="revolute">
-			<parent link="link5" />
-			<child link="link6" />
-			<origin rpy="1.571 0 0" xyz="0 -0.124 0" />
-			<axis xyz="0 0 1" />
-			<limit effort="50" lower="-6.2832" upper="6.2832" velocity="3.927"/>
-			<dynamics friction="0" />
-		</joint>
-		<link name="link6">
-			<inertial>
-				<mass value="1.16"/>
-				<origin xyz="-0.000292       7e-06     -0.0539"/>
-				<inertia ixx="0.0048282" ixy="4.1298e-06" ixz="6.9879e-06" iyy="0.0059519"
-					iyz="4.252e-06"
-					izz="0.0061263"/>
-			</inertial>
-			<visual>
-				<origin rpy="0 0 0" xyz="0 0 0" />
-				<geometry>
-					<mesh filename="package://dsr_description/meshes/m1013_white/MF1013_6_0.dae" scale="0.001 0.001 0.001" />
-				</geometry>
-			</visual>
-		</link>
-		<xacro:dsr_transmission />
-		<xacro:dsr_gazebo namespace="${namespace}" />
-	</xacro:macro>
+      <visual>
+        <origin rpy="0 0 0" xyz="0 0 0" />
+        <geometry>
+          <mesh filename="package://dsr_description/meshes/m1013_white/MF1013_5_0.dae" scale="0.001 0.001 0.001" />
+        </geometry>
+      </visual>
+    </link>
+    <!-- joint6 -->
+    <joint name="joint6" type="revolute">
+      <parent link="link5" />
+      <child link="link6" />
+      <origin rpy="1.571 0 0" xyz="0 -0.124 0" />
+      <axis xyz="0 0 1" />
+      <limit effort="50" lower="-6.2832" upper="6.2832" velocity="3.927"/>
+      <dynamics friction="0" />
+    </joint>
+    <link name="link6">
+      <inertial>
+        <mass value="1.16"/>
+        <origin xyz="-0.000292       7e-06     -0.0539"/>
+        <inertia ixx="0.0048282" ixy="4.1298e-06" ixz="6.9879e-06" iyy="0.0059519"
+          iyz="4.252e-06"
+          izz="0.0061263"/>
+      </inertial>
+      <visual>
+        <origin rpy="0 0 0" xyz="0 0 0" />
+        <geometry>
+          <mesh filename="package://dsr_description/meshes/m1013_white/MF1013_6_0.dae" scale="0.001 0.001 0.001" />
+        </geometry>
+      </visual>
+    </link>
+    <xacro:dsr_transmission />
+    <xacro:dsr_gazebo namespace="${namespace}" />
+  </xacro:macro>
 </robot>
