Commit message: Made whitespaces/tab indent consistent

File: dsr_description/xacro/macro.m1013.white.xacro (robot description, xacro)
@@ -1,210 +1,197 @@
 <?xml version="1.0"?>
-<robot name="m1013" xmlns:xacro="http://www.ros.org/wiki/xacro">
-	<xacro:include filename="$(find dsr_description)/config/macro.gazebo.xacro" />
-	<xacro:include filename="$(find dsr_description)/config/macro.transmission.xacro" />
-	<xacro:include filename="$(find dsr_description)/config/macro.materials.xacro" />
-	<xacro:macro name="m1013" params="namespace">
-		<xacro:dsr_materials />
-		<link name="base_0">
-			<inertial>
-				<mass value="4.12"/>
-				<origin xyz="-3.4e-05   -0.004815    0.048482"/>
-				<inertia ixx="0.016331" ixy="-6.4837e-06" ixz="2.0048e-06" iyy="0.014945"
-					iyz="-0.00051686"
-					izz="0.022577"/>
-			</inertial>
-			<visual>
-				<origin rpy="0 0 0" xyz="0 0 0" />
-				<geometry>
-					<mesh filename="package://dsr_description/meshes/m1013_white/MF1013_0_0.dae" scale="0.001 0.001 0.001" />
-				</geometry>
-			</visual>
-		</link>
-		<!-- joint 1 -->
-		<joint name="joint1" type="revolute">
-			<parent link="base_0" />
-			<child link="link1" />
-			<origin rpy="0 0 0" xyz="0 0 0.1525" />
-			<axis xyz="0 0 1" />
-			<limit effort="346" lower="-6.2832" upper="6.2832" velocity="2.0944"/>
-			<dynamics friction="0" />
-		</joint>
-		<link name="link1">
-			<inertial>
-				<mass value="7.8"/>
-				<origin xyz="0.000119      0.0428   -0.006383"/>
-				<inertia ixx="0.04506" ixy="4.1126e-05" ixz="-5.2533e-05" iyy="0.029679"
-					iyz="-0.0019959"
-					izz="0.047056"/>
-			</inertial>
-            <collision>
-                <geometry>
-                    <cylinder radius="0.1" length="0.2"/>
-                </geometry>
-            </collision>
-			<visual>
-				<origin rpy="0 0 0" xyz="0 0 0" />
-				<geometry>
-					<mesh filename="package://dsr_description/meshes/m1013_white/MF1013_1_0.dae" scale="0.001 0.001 0.001" />
-				</geometry>
-			</visual>
-		</link>
-		<!-- joint2 -->
-		<joint name="joint2" type="revolute">
-			<parent link="link1" />
-			<child link="link2" />
-			<origin rpy="0 -1.571 -1.571" xyz="0 0.0345 0" />
-			<axis xyz="0 0 1" />
-			<limit effort="346" lower="-6.2832" upper="6.2832" velocity="2.0944"/>
-			<dynamics friction="0" />
-		</joint>
-		<link name="link2">
-			<inertial>
-				<mass value="10.83"/>
-				<origin xyz="0.25973    -5.3e-05     0.15782"/>
-				<inertia ixx="0.037586" ixy="-0.00036999" ixz="-0.0069927" iyy="0.84943"
-					iyz="4.0201e-05"
-					izz="0.85021"/>
-			</inertial>
-            <collision>
-                <origin rpy="0 -1.571 0" xyz="0.3 0 0.1525" />
-                <geometry>
-                    <cylinder radius="0.08" length="0.75"/>
-                </geometry>
-            </collision>
-			<visual>
-				<origin rpy="0 0 0" xyz="0 0 0" />
-				<geometry>
-					<mesh filename="package://dsr_description/meshes/m1013_white/MF1013_2_0.dae" scale="0.001 0.001 0.001" />
-				</geometry>
-			</visual>
-			<visual>
-				<origin rpy="0 0 0" xyz="0 0 0" />
-				<geometry>
-					<mesh filename="package://dsr_description/meshes/m1013_white/MF1013_2_1.dae" scale="0.001 0.001 0.001" />
-				</geometry>
-			</visual>
-			<visual>
-				<origin rpy="0 0 0" xyz="0 0 0" />
-				<geometry>
-					<mesh filename="package://dsr_description/meshes/m1013_white/MF1013_2_2.dae" scale="0.001 0.001 0.001" />
-				</geometry>
-			</visual>
-		</link>
-		<!-- joint3 -->
-		<joint name="joint3" type="revolute">
-			<parent link="link2" />
-			<child link="link3" />
-			<origin rpy="0 0 1.571" xyz="0.62 0 0" />
-			<axis xyz="0 0 1" />
-			<limit effort="163" lower="-2.7925" upper="2.7925" velocity="3.1416"/>
-			<dynamics friction="0" />
-		</joint>
-		<link name="link3">
-			<inertial>
-				<mass value="3.68"/>
-				<origin xyz="-1.5e-05   -0.006702    0.044608"/>
-				<inertia ixx="0.018748" ixy="7.8071e-06" ixz="-5.0324e-06" iyy="0.018972"
-					iyz="-0.00099342"
-					izz="0.011502"/>
-			</inertial>
-            <visual>
-				<origin rpy="0 0 0" xyz="0 0 0" />
-				<geometry>
-					<mesh filename="package://dsr_description/meshes/m1013_white/MF1013_3_0.dae" scale="0.001 0.001 0.001" />
-				</geometry>
-			</visual>
-		</link>
-		<!-- joint4 -->
-		<joint name="joint4" type="revolute">
-			<parent link="link3" />
-			<child link="link4" />
-			<origin rpy="1.571 0 0" xyz="0 -0.559 0" />
-			<axis xyz="0 0 1" />
-			<limit effort="50" lower="-6.2832" upper="6.2832" velocity="3.927"/>
-			<dynamics friction="0" />
-		</joint>
-		<link name="link4">
-			<inertial>
-				<mass value="3.82"/>
-				<origin xyz="7.1e-05    0.091879    -0.18252"/>
-				<inertia ixx="0.19063" ixy="-1.8037e-05" ixz="-3.8576e-05" iyy="0.17268" iyz="-0.052996"
-					izz="0.030386"/>
-			</inertial>
-            <collision>
-                <origin rpy="-0.55 0 0" xyz="0 0.07 -0.3" />
-                <geometry>
-                    <cylinder radius="0.07" length="0.4"/>
-                </geometry>
-            </collision>
-			<visual>
-				<origin rpy="0 0 0" xyz="0 0 0" />
-				<geometry>
-					<mesh filename="package://dsr_description/meshes/m1013_white/MF1013_4_0.dae" scale="0.001 0.001 0.001" />
-				</geometry>
-			</visual>
-			<visual>
-				<origin rpy="0 0 0" xyz="0 0 0" />
-				<geometry>
-					<mesh filename="package://dsr_description/meshes/m1013_white/MF1013_4_1.dae" scale="0.001 0.001 0.001" />
-				</geometry>
-			</visual>
-		</link>
-		<!-- joint5 -->
-		<joint name="joint5" type="revolute">
-			<parent link="link4" />
-			<child link="link5" />
-			<origin rpy="-1.571 0 0" xyz="0 0 0" />
-			<axis xyz="0 0 1" />
-			<limit effort="50" lower="-6.2832" upper="6.2832" velocity="3.927"/>
-			<dynamics friction="0" />
-		</joint>
-		<link name="link5">
-			<inertial>
-				<mass value="2.82"/>
-				<origin xyz="-0.000273    0.003651    0.032088"/>
-				<inertia ixx="0.015583" ixy="2.135e-05" ixz="-5.1895e-06" iyy="0.011519"
-					iyz="0.00042553"
-					izz="0.0088671"/>
-			</inertial>
-            <collision>
-                <origin rpy="1.571 0 0" xyz="0 0 0" />
-                <geometry>
-                    <cylinder radius="0.08" length="0.15"/>
-                </geometry>
-            </collision>
-			<visual>
-				<origin rpy="0 0 0" xyz="0 0 0" />
-				<geometry>
-					<mesh filename="package://dsr_description/meshes/m1013_white/MF1013_5_0.dae" scale="0.001 0.001 0.001" />
-				</geometry>
-			</visual>
-		</link>
-		<!-- joint6 -->
-		<joint name="joint6" type="revolute">
-			<parent link="link5" />
-			<child link="link6" />
-			<origin rpy="1.571 0 0" xyz="0 -0.121 0" />
-			<axis xyz="0 0 1" />
-			<limit effort="50" lower="-6.2832" upper="6.2832" velocity="3.927"/>
-			<dynamics friction="0" />
-		</joint>
-		<link name="link6">
-			<inertial>
-				<mass value="1.16"/>
-				<origin xyz="-0.000292       7e-06     -0.0539"/>
-				<inertia ixx="0.0048282" ixy="4.1298e-06" ixz="6.9879e-06" iyy="0.0059519"
-					iyz="4.252e-06"
-					izz="0.0061263"/>
-			</inertial>
-			<visual>
-				<origin rpy="0 0 0" xyz="0 0 0" />
-				<geometry>
-					<mesh filename="package://dsr_description/meshes/m1013_white/MF1013_6_0.dae" scale="0.001 0.001 0.001" />
-				</geometry>
-			</visual>
-		</link>
-		<xacro:dsr_transmission />
-		<xacro:dsr_gazebo namespace="${namespace}" />
-	</xacro:macro>
+<robot xmlns:xacro="http://www.ros.org/wiki/xacro" name="m1013">
+  <xacro:include filename="$(find dsr_description)/config/macro.gazebo.xacro"/>
+  <xacro:include filename="$(find dsr_description)/config/macro.transmission.xacro"/>
+  <xacro:include filename="$(find dsr_description)/config/macro.materials.xacro"/>
+  <xacro:macro name="m1013" params="namespace">
+    <xacro:dsr_materials/>
+    <link name="base_0">
+      <inertial>
+        <mass value="4.12"/>
+        <origin xyz="-3.4e-05   -0.004815    0.048482"/>
+        <inertia ixx="0.016331" ixy="-6.4837e-06" ixz="2.0048e-06" iyy="0.014945" iyz="-0.00051686" izz="0.022577"/>
+      </inertial>
+      <visual>
+        <origin rpy="0 0 0" xyz="0 0 0"/>
+        <geometry>
+          <mesh filename="package://dsr_description/meshes/m1013_white/MF1013_0_0.dae" scale="0.001 0.001 0.001"/>
+        </geometry>
+      </visual>
+    </link>
+    <!-- joint 1 -->
+    <joint name="joint1" type="revolute">
+      <parent link="base_0"/>
+      <child link="link1"/>
+      <origin rpy="0 0 0" xyz="0 0 0.1525"/>
+      <axis xyz="0 0 1"/>
+      <limit effort="346" lower="-6.2832" upper="6.2832" velocity="2.0944"/>
+      <dynamics friction="0"/>
+    </joint>
+    <link name="link1">
+      <inertial>
+        <mass value="7.8"/>
+        <origin xyz="0.000119      0.0428   -0.006383"/>
+        <inertia ixx="0.04506" ixy="4.1126e-05" ixz="-5.2533e-05" iyy="0.029679" iyz="-0.0019959" izz="0.047056"/>
+      </inertial>
+      <collision>
+        <geometry>
+          <cylinder radius="0.1" length="0.2"/>
+        </geometry>
+      </collision>
+      <visual>
+        <origin rpy="0 0 0" xyz="0 0 0"/>
+        <geometry>
+          <mesh filename="package://dsr_description/meshes/m1013_white/MF1013_1_0.dae" scale="0.001 0.001 0.001"/>
+        </geometry>
+      </visual>
+    </link>
+    <!-- joint2 -->
+    <joint name="joint2" type="revolute">
+      <parent link="link1"/>
+      <child link="link2"/>
+      <origin rpy="0 -1.571 -1.571" xyz="0 0.0345 0"/>
+      <axis xyz="0 0 1"/>
+      <limit effort="346" lower="-6.2832" upper="6.2832" velocity="2.0944"/>
+      <dynamics friction="0"/>
+    </joint>
+    <link name="link2">
+      <inertial>
+        <mass value="10.83"/>
+        <origin xyz="0.25973    -5.3e-05     0.15782"/>
+        <inertia ixx="0.037586" ixy="-0.00036999" ixz="-0.0069927" iyy="0.84943" iyz="4.0201e-05" izz="0.85021"/>
+      </inertial>
+      <collision>
+        <origin rpy="0 -1.571 0" xyz="0.3 0 0.1525"/>
+        <geometry>
+          <cylinder radius="0.08" length="0.75"/>
+        </geometry>
+      </collision>
+      <visual>
+        <origin rpy="0 0 0" xyz="0 0 0"/>
+        <geometry>
+          <mesh filename="package://dsr_description/meshes/m1013_white/MF1013_2_0.dae" scale="0.001 0.001 0.001"/>
+        </geometry>
+      </visual>
+      <visual>
+        <origin rpy="0 0 0" xyz="0 0 0"/>
+        <geometry>
+          <mesh filename="package://dsr_description/meshes/m1013_white/MF1013_2_1.dae" scale="0.001 0.001 0.001"/>
+        </geometry>
+      </visual>
+      <visual>
+        <origin rpy="0 0 0" xyz="0 0 0"/>
+        <geometry>
+          <mesh filename="package://dsr_description/meshes/m1013_white/MF1013_2_2.dae" scale="0.001 0.001 0.001"/>
+        </geometry>
+      </visual>
+    </link>
+    <!-- joint3 -->
+    <joint name="joint3" type="revolute">
+      <parent link="link2"/>
+      <child link="link3"/>
+      <origin rpy="0 0 1.571" xyz="0.62 0 0"/>
+      <axis xyz="0 0 1"/>
+      <limit effort="163" lower="-2.7925" upper="2.7925" velocity="3.1416"/>
+      <dynamics friction="0"/>
+    </joint>
+    <link name="link3">
+      <inertial>
+        <mass value="3.68"/>
+        <origin xyz="-1.5e-05   -0.006702    0.044608"/>
+        <inertia ixx="0.018748" ixy="7.8071e-06" ixz="-5.0324e-06" iyy="0.018972" iyz="-0.00099342" izz="0.011502"/>
+      </inertial>
+      <visual>
+        <origin rpy="0 0 0" xyz="0 0 0"/>
+        <geometry>
+          <mesh filename="package://dsr_description/meshes/m1013_white/MF1013_3_0.dae" scale="0.001 0.001 0.001"/>
+        </geometry>
+      </visual>
+    </link>
+    <!-- joint4 -->
+    <joint name="joint4" type="revolute">
+      <parent link="link3"/>
+      <child link="link4"/>
+      <origin rpy="1.571 0 0" xyz="0 -0.559 0"/>
+      <axis xyz="0 0 1"/>
+      <limit effort="50" lower="-6.2832" upper="6.2832" velocity="3.927"/>
+      <dynamics friction="0"/>
+    </joint>
+    <link name="link4">
+      <inertial>
+        <mass value="3.82"/>
+        <origin xyz="7.1e-05    0.091879    -0.18252"/>
+        <inertia ixx="0.19063" ixy="-1.8037e-05" ixz="-3.8576e-05" iyy="0.17268" iyz="-0.052996" izz="0.030386"/>
+      </inertial>
+      <collision>
+        <origin rpy="-0.55 0 0" xyz="0 0.07 -0.3"/>
+        <geometry>
+          <cylinder radius="0.07" length="0.4"/>
+        </geometry>
+      </collision>
+      <visual>
+        <origin rpy="0 0 0" xyz="0 0 0"/>
+        <geometry>
+          <mesh filename="package://dsr_description/meshes/m1013_white/MF1013_4_0.dae" scale="0.001 0.001 0.001"/>
+        </geometry>
+      </visual>
+      <visual>
+        <origin rpy="0 0 0" xyz="0 0 0"/>
+        <geometry>
+          <mesh filename="package://dsr_description/meshes/m1013_white/MF1013_4_1.dae" scale="0.001 0.001 0.001"/>
+        </geometry>
+      </visual>
+    </link>
+    <!-- joint5 -->
+    <joint name="joint5" type="revolute">
+      <parent link="link4"/>
+      <child link="link5"/>
+      <origin rpy="-1.571 0 0" xyz="0 0 0"/>
+      <axis xyz="0 0 1"/>
+      <limit effort="50" lower="-6.2832" upper="6.2832" velocity="3.927"/>
+      <dynamics friction="0"/>
+    </joint>
+    <link name="link5">
+      <inertial>
+        <mass value="2.82"/>
+        <origin xyz="-0.000273    0.003651    0.032088"/>
+        <inertia ixx="0.015583" ixy="2.135e-05" ixz="-5.1895e-06" iyy="0.011519" iyz="0.00042553" izz="0.0088671"/>
+      </inertial>
+      <collision>
+        <origin rpy="1.571 0 0" xyz="0 0 0"/>
+        <geometry>
+          <cylinder radius="0.08" length="0.15"/>
+        </geometry>
+      </collision>
+      <visual>
+        <origin rpy="0 0 0" xyz="0 0 0"/>
+        <geometry>
+          <mesh filename="package://dsr_description/meshes/m1013_white/MF1013_5_0.dae" scale="0.001 0.001 0.001"/>
+        </geometry>
+      </visual>
+    </link>
+    <!-- joint6 -->
+    <joint name="joint6" type="revolute">
+      <parent link="link5"/>
+      <child link="link6"/>
+      <origin rpy="1.571 0 0" xyz="0 -0.121 0"/>
+      <axis xyz="0 0 1"/>
+      <limit effort="50" lower="-6.2832" upper="6.2832" velocity="3.927"/>
+      <dynamics friction="0"/>
+    </joint>
+    <link name="link6">
+      <inertial>
+        <mass value="1.16"/>
+        <origin xyz="-0.000292       7e-06     -0.0539"/>
+        <inertia ixx="0.0048282" ixy="4.1298e-06" ixz="6.9879e-06" iyy="0.0059519" iyz="4.252e-06" izz="0.0061263"/>
+      </inertial>
+      <visual>
+        <origin rpy="0 0 0" xyz="0 0 0"/>
+        <geometry>
+          <mesh filename="package://dsr_description/meshes/m1013_white/MF1013_6_0.dae" scale="0.001 0.001 0.001"/>
+        </geometry>
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
Commit message: Added collision model for m1013.white (reduced stl)

File: dsr_description/xacro/macro.m1013.white.xacro (robot description, xacro)
@@ -15,9 +15,14 @@
       </inertial>
       <visual>
-        <origin rpy="0 0 0" xyz="0 0 0" />
+        <material name="dr_gray" />
         <geometry>
           <mesh filename="package://dsr_description/meshes/m1013_white/MF1013_0_0.dae" scale="0.001 0.001 0.001" />
         </geometry>
       </visual>
+      <collision>
+        <geometry>
+          <mesh filename="package://dsr_description/meshes/m1013_collision/MF1013_0_0.stl" scale="0.001 0.001 0.001" />
+        </geometry>
+      </collision>
     </link>
     <!-- joint 1 -->
@@ -38,15 +43,15 @@
           izz="0.047056"/>
       </inertial>
-      <collision>
-        <geometry>
-          <cylinder radius="0.1" length="0.2"/>
-        </geometry>
-      </collision>
-      <visual>
-        <origin rpy="0 0 0" xyz="0 0 0" />
+      <visual>
+        <material name="dr_white" />
         <geometry>
           <mesh filename="package://dsr_description/meshes/m1013_white/MF1013_1_0.dae" scale="0.001 0.001 0.001" />
         </geometry>
       </visual>
+      <collision>
+        <geometry>
+          <mesh filename="package://dsr_description/meshes/m1013_collision/MF1013_1_0.stl" scale="0.001 0.001 0.001" />
+        </geometry>
+      </collision>
     </link>
     <!-- joint2 -->
@@ -67,28 +72,35 @@
           izz="0.85021"/>
       </inertial>
-            <collision>
-                <origin rpy="0 -1.571 0" xyz="0.3 0 0.1525" />
-                <geometry>
-                    <cylinder radius="0.08" length="0.75"/>
-                </geometry>
-            </collision>
-      <visual>
-        <origin rpy="0 0 0" xyz="0 0 0" />
+      <visual>
+        <material name="dr_white" />
         <geometry>
           <mesh filename="package://dsr_description/meshes/m1013_white/MF1013_2_0.dae" scale="0.001 0.001 0.001" />
         </geometry>
       </visual>
-      <visual>
-        <origin rpy="0 0 0" xyz="0 0 0" />
+      <collision>
+        <geometry>
+          <mesh filename="package://dsr_description/meshes/m1013_collision/MF1013_2_0.stl" scale="0.001 0.001 0.001" />
+        </geometry>
+      </collision>
+      <visual>
         <geometry>
           <mesh filename="package://dsr_description/meshes/m1013_white/MF1013_2_1.dae" scale="0.001 0.001 0.001" />
         </geometry>
       </visual>
-      <visual>
-        <origin rpy="0 0 0" xyz="0 0 0" />
+      <collision>
+        <geometry>
+          <mesh filename="package://dsr_description/meshes/m1013_collision/MF1013_2_1.stl" scale="0.001 0.001 0.001" />
+        </geometry>
+      </collision>
+      <visual>
         <geometry>
           <mesh filename="package://dsr_description/meshes/m1013_white/MF1013_2_2.dae" scale="0.001 0.001 0.001" />
         </geometry>
       </visual>
+      <collision>
+        <geometry>
+          <mesh filename="package://dsr_description/meshes/m1013_collision/MF1013_2_2.stl" scale="0.001 0.001 0.001" />
+        </geometry>
+      </collision>
     </link>
     <!-- joint3 -->
@@ -109,10 +121,15 @@
           izz="0.011502"/>
       </inertial>
-            <visual>
-        <origin rpy="0 0 0" xyz="0 0 0" />
+      <visual>
+        <material name="dr_white" />
         <geometry>
           <mesh filename="package://dsr_description/meshes/m1013_white/MF1013_3_0.dae" scale="0.001 0.001 0.001" />
         </geometry>
       </visual>
+      <collision>
+        <geometry>
+          <mesh filename="package://dsr_description/meshes/m1013_collision/MF1013_3_0.stl" scale="0.001 0.001 0.001" />
+        </geometry>
+      </collision>
     </link>
     <!-- joint4 -->
@@ -132,22 +149,25 @@
           izz="0.030386"/>
       </inertial>
-            <collision>
-                <origin rpy="-0.55 0 0" xyz="0 0.07 -0.3" />
-                <geometry>
-                    <cylinder radius="0.07" length="0.4"/>
-                </geometry>
-            </collision>
-      <visual>
-        <origin rpy="0 0 0" xyz="0 0 0" />
+      <visual>
+        <material name="dr_white" />
         <geometry>
           <mesh filename="package://dsr_description/meshes/m1013_white/MF1013_4_0.dae" scale="0.001 0.001 0.001" />
         </geometry>
       </visual>
-      <visual>
-        <origin rpy="0 0 0" xyz="0 0 0" />
+      <collision>
+        <geometry>
+          <mesh filename="package://dsr_description/meshes/m1013_collision/MF1013_4_0.stl" scale="0.001 0.001 0.001" />
+        </geometry>
+      </collision>
+      <visual>
         <geometry>
           <mesh filename="package://dsr_description/meshes/m1013_white/MF1013_4_1.dae" scale="0.001 0.001 0.001" />
         </geometry>
       </visual>
+      <collision>
+        <geometry>
+          <mesh filename="package://dsr_description/meshes/m1013_collision/MF1013_4_1.stl" scale="0.001 0.001 0.001" />
+        </geometry>
+      </collision>
     </link>
     <!-- joint5 -->
@@ -168,16 +188,15 @@
           izz="0.0088671"/>
       </inertial>
-            <collision>
-                <origin rpy="1.571 0 0" xyz="0 0 0" />
-                <geometry>
-                    <cylinder radius="0.08" length="0.15"/>
-                </geometry>
-            </collision>
-      <visual>
-        <origin rpy="0 0 0" xyz="0 0 0" />
+      <visual>
+        <material name="dr_white" />
         <geometry>
           <mesh filename="package://dsr_description/meshes/m1013_white/MF1013_5_0.dae" scale="0.001 0.001 0.001" />
         </geometry>
       </visual>
+      <collision>
+        <geometry>
+          <mesh filename="package://dsr_description/meshes/m1013_collision/MF1013_5_0.stl" scale="0.001 0.001 0.001" />
+        </geometry>
+      </collision>
     </link>
     <!-- joint6 -->
@@ -199,9 +218,14 @@
       </inertial>
       <visual>
-        <origin rpy="0 0 0" xyz="0 0 0" />
+        <material name="dr_gray" />
         <geometry>
           <mesh filename="package://dsr_description/meshes/m1013_white/MF1013_6_0.dae" scale="0.001 0.001 0.001" />
         </geometry>
       </visual>
+      <collision>
+        <geometry>
+          <mesh filename="package://dsr_description/meshes/m1013_collision/MF1013_6_0.stl" scale="0.001 0.001 0.001" />
+        </geometry>
+      </collision>
     </link>
     <xacro:dsr_transmission />
