Commit message: Added collision model for m1013.white (reduced stl)

File: dsr_description/xacro/macro.m1013.white.xacro (robot description, xacro)
@@ -13,9 +13,14 @@
       </inertial>
       <visual>
-        <origin rpy="0 0 0" xyz="0 0 0"/>
+        <material name="dr_gray"/>
         <geometry>
           <mesh filename="package://dsr_description/meshes/m1013_white/MF1013_0_0.dae" scale="0.001 0.001 0.001"/>
         </geometry>
       </visual>
+      <collision>
+        <geometry>
+          <mesh filename="package://dsr_description/meshes/m1013_collision/MF1013_0_0.stl" scale="0.001 0.001 0.001"/>
+        </geometry>
+      </collision>
     </link>
     <!-- joint 1 -->
@@ -34,15 +39,15 @@
         <inertia ixx="0.04506" ixy="4.1126e-05" ixz="-5.2533e-05" iyy="0.029679" iyz="-0.0019959" izz="0.047056"/>
       </inertial>
-      <collision>
-        <geometry>
-          <cylinder radius="0.1" length="0.2"/>
-        </geometry>
-      </collision>
-      <visual>
-        <origin rpy="0 0 0" xyz="0 0 0"/>
+      <visual>
+        <material name="dr_white"/>
         <geometry>
           <mesh filename="package://dsr_description/meshes/m1013_white/MF1013_1_0.dae" scale="0.001 0.001 0.001"/>
         </geometry>
       </visual>
+      <collision>
+        <geometry>
+          <mesh filename="package://dsr_description/meshes/m1013_collision/MF1013_1_0.stl" scale="0.001 0.001 0.001"/>
+        </geometry>
+      </collision>
     </link>
     <!-- joint2 -->
@@ -61,28 +66,35 @@
         <inertia ixx="0.037586" ixy="-0.00036999" ixz="-0.0069927" iyy="0.84943" iyz="4.0201e-05" izz="0.85021"/>
       </inertial>
-      <collision>
-        <origin rpy="0 -1.571 0" xyz="0.3 0 0.1525"/>
-        <geometry>
-          <cylinder radius="0.08" length="0.75"/>
-        </geometry>
-      </collision>
-      <visual>
-        <origin rpy="0 0 0" xyz="0 0 0"/>
+      <visual>
+        <material name="dr_white"/>
         <geometry>
           <mesh filename="package://dsr_description/meshes/m1013_white/MF1013_2_0.dae" scale="0.001 0.001 0.001"/>
         </geometry>
       </visual>
-      <visual>
-        <origin rpy="0 0 0" xyz="0 0 0"/>
+      <collision>
+        <geometry>
+          <mesh filename="package://dsr_description/meshes/m1013_collision/MF1013_2_0.stl" scale="0.001 0.001 0.001"/>
+        </geometry>
+      </collision>
+      <visual>
         <geometry>
           <mesh filename="package://dsr_description/meshes/m1013_white/MF1013_2_1.dae" scale="0.001 0.001 0.001"/>
         </geometry>
       </visual>
-      <visual>
-        <origin rpy="0 0 0" xyz="0 0 0"/>
+      <collision>
+        <geometry>
+          <mesh filename="package://dsr_description/meshes/m1013_collision/MF1013_2_1.stl" scale="0.001 0.001 0.001"/>
+        </geometry>
+      </collision>
+      <visual>
         <geometry>
           <mesh filename="package://dsr_description/meshes/m1013_white/MF1013_2_2.dae" scale="0.001 0.001 0.001"/>
         </geometry>
       </visual>
+      <collision>
+        <geometry>
+          <mesh filename="package://dsr_description/meshes/m1013_collision/MF1013_2_2.stl" scale="0.001 0.001 0.001"/>
+        </geometry>
+      </collision>
     </link>
     <!-- joint3 -->
@@ -102,9 +114,14 @@
       </inertial>
       <visual>
-        <origin rpy="0 0 0" xyz="0 0 0"/>
+        <material name="dr_white"/>
         <geometry>
           <mesh filename="package://dsr_description/meshes/m1013_white/MF1013_3_0.dae" scale="0.001 0.001 0.001"/>
         </geometry>
       </visual>
+      <collision>
+        <geometry>
+          <mesh filename="package://dsr_description/meshes/m1013_collision/MF1013_3_0.stl" scale="0.001 0.001 0.001"/>
+        </geometry>
+      </collision>
     </link>
     <!-- joint4 -->
@@ -123,22 +140,25 @@
         <inertia ixx="0.19063" ixy="-1.8037e-05" ixz="-3.8576e-05" iyy="0.17268" iyz="-0.052996" izz="0.030386"/>
       </inertial>
-      <collision>
-        <origin rpy="-0.55 0 0" xyz="0 0.07 -0.3"/>
-        <geometry>
-          <cylinder radius="0.07" length="0.4"/>
-        </geometry>
-      </collision>
-      <visual>
-        <origin rpy="0 0 0" xyz="0 0 0"/>
+      <visual>
+        <material name="dr_white"/>
         <geometry>
           <mesh filename="package://dsr_description/meshes/m1013_white/MF1013_4_0.dae" scale="0.001 0.001 0.001"/>
         </geometry>
       </visual>
-      <visual>
-        <origin rpy="0 0 0" xyz="0 0 0"/>
+      <collision>
+        <geometry>
+          <mesh filename="package://dsr_description/meshes/m1013_collision/MF1013_4_0.stl" scale="0.001 0.001 0.001"/>
+        </geometry>
+      </collision>
+      <visual>
         <geometry>
           <mesh filename="package://dsr_description/meshes/m1013_white/MF1013_4_1.dae" scale="0.001 0.001 0.001"/>
         </geometry>
       </visual>
+      <collision>
+        <geometry>
+          <mesh filename="package://dsr_description/meshes/m1013_collision/MF1013_4_1.stl" scale="0.001 0.001 0.001"/>
+        </geometry>
+      </collision>
     </link>
     <!-- joint5 -->
@@ -157,16 +177,15 @@
         <inertia ixx="0.015583" ixy="2.135e-05" ixz="-5.1895e-06" iyy="0.011519" iyz="0.00042553" izz="0.0088671"/>
       </inertial>
-      <collision>
-        <origin rpy="1.571 0 0" xyz="0 0 0"/>
-        <geometry>
-          <cylinder radius="0.08" length="0.15"/>
-        </geometry>
-      </collision>
-      <visual>
-        <origin rpy="0 0 0" xyz="0 0 0"/>
+      <visual>
+        <material name="dr_white"/>
         <geometry>
           <mesh filename="package://dsr_description/meshes/m1013_white/MF1013_5_0.dae" scale="0.001 0.001 0.001"/>
         </geometry>
       </visual>
+      <collision>
+        <geometry>
+          <mesh filename="package://dsr_description/meshes/m1013_collision/MF1013_5_0.stl" scale="0.001 0.001 0.001"/>
+        </geometry>
+      </collision>
     </link>
     <!-- joint6 -->
@@ -186,9 +205,14 @@
       </inertial>
       <visual>
-        <origin rpy="0 0 0" xyz="0 0 0"/>
+        <material name="dr_gray"/>
         <geometry>
           <mesh filename="package://dsr_description/meshes/m1013_white/MF1013_6_0.dae" scale="0.001 0.001 0.001"/>
         </geometry>
       </visual>
+      <collision>
+        <geometry>
+          <mesh filename="package://dsr_description/meshes/m1013_collision/MF1013_6_0.stl" scale="0.001 0.001 0.001"/>
+        </geometry>
+      </collision>
     </link>
     <xacro:dsr_transmission/>
