Commit message: Use opw IK solver for m1013
- use 0.121 instead of 0.124 for z-offset of joint6
- use constant 'pi' for xacro joint rotations to avoid error with FK test of opw

File: dsr_description/xacro/macro.m1013.blue.xacro (robot description, xacro)
@@ -54,5 +54,5 @@
 			<parent link="link1" />
 			<child link="link2" />
-			<origin rpy="0 -1.571 -1.571" xyz="0 0.0345 0" />
+			<origin rpy="0 -${pi/2} -${pi/2}" xyz="0 0.0345 0" />
 			<axis xyz="0 0 1" />
 			<limit effort="346" lower="-6.2832" upper="6.2832" velocity="2.0944"/>
@@ -96,5 +96,5 @@
 			<parent link="link2" />
 			<child link="link3" />
-			<origin rpy="0 0 1.571" xyz="0.62 0 0" />
+			<origin rpy="0 0 ${pi/2}" xyz="0.62 0 0" />
 			<axis xyz="0 0 1" />
 			<limit effort="163" lower="-2.7925" upper="2.7925" velocity="3.1416"/>
@@ -120,5 +120,5 @@
 			<parent link="link3" />
 			<child link="link4" />
-			<origin rpy="1.571 0 0" xyz="0 -0.559 0" />
+			<origin rpy="${pi/2} 0 0" xyz="0 -0.559 0" />
 			<axis xyz="0 0 1" />
 			<limit effort="50" lower="-6.2832" upper="6.2832" velocity="3.927"/>
@@ -155,5 +155,5 @@
 			<parent link="link4" />
 			<child link="link5" />
-			<origin rpy="-1.571 0 0" xyz="0 0 0" />
+			<origin rpy="-${pi/2} 0 0" xyz="0 0 0" />
 			<axis xyz="0 0 1" />
 			<limit effort="50" lower="-6.2832" upper="6.2832" velocity="3.927"/>
@@ -185,5 +185,5 @@
 			<parent link="link5" />
 			<child link="link6" />
-			<origin rpy="1.571 0 0" xyz="0 -0.121 0" />
+			<origin rpy="${pi/2} 0 0" xyz="0 -0.121 0" />
 			<axis xyz="0 0 1" />
 			<limit effort="50" lower="-6.2832" upper="6.2832" velocity="3.927"/>

File: dsr_description/xacro/macro.m1013.white.xacro (robot description, xacro)
@@ -55,5 +55,5 @@
       <parent link="link1"/>
       <child link="link2"/>
-      <origin rpy="0 -1.571 -1.571" xyz="0 0.0345 0"/>
+      <origin rpy="0 -${pi/2} -${pi/2}" xyz="0 0.0345 0"/>
       <axis xyz="0 0 1"/>
       <limit effort="346" lower="-6.2832" upper="6.2832" velocity="2.0944"/>
@@ -102,5 +102,5 @@
       <parent link="link2"/>
       <child link="link3"/>
-      <origin rpy="0 0 1.571" xyz="0.62 0 0"/>
+      <origin rpy="0 0 ${pi/2}" xyz="0.62 0 0"/>
       <axis xyz="0 0 1"/>
       <limit effort="163" lower="-2.7925" upper="2.7925" velocity="3.1416"/>
@@ -129,5 +129,5 @@
       <parent link="link3"/>
       <child link="link4"/>
-      <origin rpy="1.571 0 0" xyz="0 -0.559 0"/>
+      <origin rpy="${pi/2} 0 0" xyz="0 -0.559 0"/>
       <axis xyz="0 0 1"/>
       <limit effort="50" lower="-6.2832" upper="6.2832" velocity="3.927"/>
@@ -166,5 +166,5 @@
       <parent link="link4"/>
       <child link="link5"/>
-      <origin rpy="-1.571 0 0" xyz="0 0 0"/>
+      <origin rpy="-${pi/2} 0 0" xyz="0 0 0"/>
       <axis xyz="0 0 1"/>
       <limit effort="50" lower="-6.2832" upper="6.2832" velocity="3.927"/>
@@ -193,5 +193,5 @@
       <parent link="link5"/>
       <child link="link6"/>
-      <origin rpy="1.571 0 0" xyz="0 -0.121 0"/>
+      <origin rpy="${pi/2} 0 0" xyz="0 -0.121 0"/>
       <axis xyz="0 0 1"/>
       <limit effort="50" lower="-6.2832" upper="6.2832" velocity="3.927"/>

Commit message: Use opw IK solver for m1013
- use 0.121 instead of 0.124 for z-offset of joint6
- use constant 'pi' for xacro joint rotations to avoid error with FK test of opw

File: dsr_description/xacro/macro.m1013.blue.xacro (robot description, xacro)
@@ -54,5 +54,5 @@
 			<parent link="link1" />
 			<child link="link2" />
-			<origin rpy="0 -1.571 -1.571" xyz="0 0.0345 0" />
+			<origin rpy="0 -${pi/2} -${pi/2}" xyz="0 0.0345 0" />
 			<axis xyz="0 0 1" />
 			<limit effort="346" lower="-6.2832" upper="6.2832" velocity="2.0944"/>
@@ -96,5 +96,5 @@
 			<parent link="link2" />
 			<child link="link3" />
-			<origin rpy="0 0 1.571" xyz="0.62 0 0" />
+			<origin rpy="0 0 ${pi/2}" xyz="0.62 0 0" />
 			<axis xyz="0 0 1" />
 			<limit effort="163" lower="-2.7925" upper="2.7925" velocity="3.1416"/>
@@ -120,5 +120,5 @@
 			<parent link="link3" />
 			<child link="link4" />
-			<origin rpy="1.571 0 0" xyz="0 -0.559 0" />
+			<origin rpy="${pi/2} 0 0" xyz="0 -0.559 0" />
 			<axis xyz="0 0 1" />
 			<limit effort="50" lower="-6.2832" upper="6.2832" velocity="3.927"/>
@@ -155,5 +155,5 @@
 			<parent link="link4" />
 			<child link="link5" />
-			<origin rpy="-1.571 0 0" xyz="0 0 0" />
+			<origin rpy="-${pi/2} 0 0" xyz="0 0 0" />
 			<axis xyz="0 0 1" />
 			<limit effort="50" lower="-6.2832" upper="6.2832" velocity="3.927"/>
@@ -185,5 +185,5 @@
 			<parent link="link5" />
 			<child link="link6" />
-			<origin rpy="1.571 0 0" xyz="0 -0.124 0" />
+			<origin rpy="${pi/2} 0 0" xyz="0 -0.121 0" />
 			<axis xyz="0 0 1" />
 			<limit effort="50" lower="-6.2832" upper="6.2832" velocity="3.927"/>

File: dsr_description/xacro/macro.m1013.white.xacro (robot description, xacro)
@@ -59,5 +59,5 @@
       <parent link="link1" />
       <child link="link2" />
-      <origin rpy="0 -1.571 -1.571" xyz="0 0.0345 0" />
+      <origin rpy="0 -${pi/2} -${pi/2}" xyz="0 0.0345 0" />
       <axis xyz="0 0 1" />
       <limit effort="346" lower="-6.2832" upper="6.2832" velocity="2.0944"/>
@@ -108,5 +108,5 @@
       <parent link="link2" />
       <child link="link3" />
-      <origin rpy="0 0 1.571" xyz="0.62 0 0" />
+      <origin rpy="0 0 ${pi/2}" xyz="0.62 0 0" />
       <axis xyz="0 0 1" />
       <limit effort="163" lower="-2.7925" upper="2.7925" velocity="3.1416"/>
@@ -137,5 +137,5 @@
       <parent link="link3" />
       <child link="link4" />
-      <origin rpy="1.571 0 0" xyz="0 -0.559 0" />
+      <origin rpy="${pi/2} 0 0" xyz="0 -0.559 0" />
       <axis xyz="0 0 1" />
       <limit effort="50" lower="-6.2832" upper="6.2832" velocity="3.927"/>
@@ -175,5 +175,5 @@
       <parent link="link4" />
       <child link="link5" />
-      <origin rpy="-1.571 0 0" xyz="0 0 0" />
+      <origin rpy="-${pi/2} 0 0" xyz="0 0 0" />
       <axis xyz="0 0 1" />
       <limit effort="50" lower="-6.2832" upper="6.2832" velocity="3.927"/>
@@ -204,5 +204,5 @@
       <parent link="link5" />
       <child link="link6" />
-      <origin rpy="1.571 0 0" xyz="0 -0.124 0" />
+      <origin rpy="${pi/2} 0 0" xyz="0 -0.121 0" />
       <axis xyz="0 0 1" />
       <limit effort="50" lower="-6.2832" upper="6.2832" velocity="3.927"/>
