Commit message: added collision model for a0509.white (reduced stl)

File: dsr_description/xacro/macro.a0509.white.xacro (robot description, xacro)
@@ -4,7 +4,7 @@
 	<xacro:include filename="$(find dsr_description)/config/macro.transmission.xacro" />
 	<xacro:include filename="$(find dsr_description)/config/macro.materials.xacro" />
-	<xacro:macro name="a0509" params="namespace">
+	<xacro:macro name="a0509" params="prefix:='' namespace:=''">
 		<xacro:dsr_materials />
-		<link name="base_0">
+		<link name="${prefix}base_link">
 			<inertial>
 				<mass value="2.198"/>
@@ -20,8 +20,14 @@
 				</geometry>
 			</visual>
+            <collision>
+				<origin rpy="0 0 0" xyz="0 0 0" />
+				<geometry>
+					<mesh filename="package://dsr_description/meshes/a0509_collision/A0509_0_0.stl" scale="0.001 0.001 0.001" />
+				</geometry>
+			</collision>
 		</link>
 		<!-- joint 1 -->
 		<joint name="joint1" type="revolute">
-			<parent link="base_0" />
+			<parent link="base_link" />
 			<child link="link1" />
 			<origin rpy="0 0 0" xyz="0 0 0.1555" />
@@ -37,9 +43,4 @@
 					izz="0.01686"/>
 			</inertial>
-            <collision>
-                <geometry>
-                    <cylinder radius="0.08" length="0.2"/>
-                </geometry>
-            </collision>
 			<visual>
 				<origin rpy="0 0 0" xyz="0 0 0" />
@@ -48,4 +49,10 @@
 				</geometry>
 			</visual>
+            <collision>
+				<origin rpy="0 0 0" xyz="0 0 0" />
+				<geometry>
+					<mesh filename="package://dsr_description/meshes/a0509_collision/A0509_1_0.stl" scale="0.001 0.001 0.001" />
+				</geometry>
+			</collision>
             <visual>
 				<origin rpy="0 0 0" xyz="0 0 0" />
@@ -54,4 +61,10 @@
 				</geometry>
 			</visual>
+            <collision>
+				<origin rpy="0 0 0" xyz="0 0 0" />
+				<geometry>
+					<mesh filename="package://dsr_description/meshes/a0509_collision/A0509_1_1.stl" scale="0.001 0.001 0.001" />
+				</geometry>
+			</collision>
             <visual>
 				<origin rpy="0 0 0" xyz="0 0 0" />
@@ -60,4 +73,10 @@
 				</geometry>
 			</visual>
+            <collision>
+				<origin rpy="0 0 0" xyz="0 0 0" />
+				<geometry>
+					<mesh filename="package://dsr_description/meshes/a0509_collision/A0509_1_2.stl" scale="0.001 0.001 0.001" />
+				</geometry>
+			</collision>
 		</link>
 		<!-- joint2 -->
@@ -77,10 +96,4 @@
 					izz="0.25442"/>
 			</inertial>
-            <collision>
-                <origin rpy="0 -1.571 0" xyz="0.2 0 0.1525" />
-                <geometry>
-                    <cylinder radius="0.08" length="0.5"/>
-                </geometry>
-            </collision>
 			<visual>
 				<origin rpy="0 0 0" xyz="0 0 0" />
@@ -89,4 +102,10 @@
 				</geometry>
 			</visual>
+            <collision>
+				<origin rpy="0 0 0" xyz="0 0 0" />
+				<geometry>
+					<mesh filename="package://dsr_description/meshes/a0509_collision/A0509_2_0.stl" scale="0.001 0.001 0.001" />
+				</geometry>
+			</collision>
 			<visual>
 				<origin rpy="0 0 0" xyz="0 0 0" />
@@ -95,4 +114,10 @@
 				</geometry>
 			</visual>
+            <collision>
+				<origin rpy="0 0 0" xyz="0 0 0" />
+				<geometry>
+					<mesh filename="package://dsr_description/meshes/a0509_collision/A0509_2_1.stl" scale="0.001 0.001 0.001" />
+				</geometry>
+			</collision>
 			<visual>
 				<origin rpy="0 0 0" xyz="0 0 0" />
@@ -101,4 +126,10 @@
 				</geometry>
 			</visual>
+            <collision>
+				<origin rpy="0 0 0" xyz="0 0 0" />
+				<geometry>
+					<mesh filename="package://dsr_description/meshes/a0509_collision/A0509_2_2.stl" scale="0.001 0.001 0.001" />
+				</geometry>
+			</collision>
 		</link>
 		<!-- joint3 -->
@@ -125,4 +156,10 @@
 				</geometry>
 			</visual>
+            <collision>
+				<origin rpy="0 0 0" xyz="0 0 0" />
+				<geometry>
+					<mesh filename="package://dsr_description/meshes/a0509_collision/A0509_3_0.stl" scale="0.001 0.001 0.001" />
+				</geometry>
+			</collision>
             <visual>
 				<origin rpy="0 0 0" xyz="0 0 0" />
@@ -131,4 +168,10 @@
 				</geometry>
 			</visual>
+            <collision>
+				<origin rpy="0 0 0" xyz="0 0 0" />
+				<geometry>
+					<mesh filename="package://dsr_description/meshes/a0509_collision/A0509_3_1.stl" scale="0.001 0.001 0.001" />
+				</geometry>
+			</collision>
 		</link>
 		<!-- joint4 -->
@@ -148,10 +191,4 @@
 					izz="0.013329"/>
 			</inertial>
-            <collision>
-                <origin rpy="-0.55 0 0" xyz="0 0.05 -0.2" />
-                <geometry>
-                    <cylinder radius="0.05" length="0.4"/>
-                </geometry>
-            </collision>
 			<visual>
 				<origin rpy="0 0 0" xyz="0 0 0" />
@@ -160,4 +197,10 @@
 				</geometry>
 			</visual>
+            <collision>
+				<origin rpy="0 0 0" xyz="0 0 0" />
+				<geometry>
+					<mesh filename="package://dsr_description/meshes/a0509_collision/A0509_4_0.stl" scale="0.001 0.001 0.001" />
+				</geometry>
+			</collision>
 			<visual>
 				<origin rpy="0 0 0" xyz="0 0 0" />
@@ -166,4 +209,10 @@
 				</geometry>
 			</visual>
+            <collision>
+				<origin rpy="0 0 0" xyz="0 0 0" />
+				<geometry>
+					<mesh filename="package://dsr_description/meshes/a0509_collision/A0509_4_1.stl" scale="0.001 0.001 0.001" />
+				</geometry>
+			</collision>
 		</link>
 		<!-- joint5 -->
@@ -184,10 +233,4 @@
 					izz="0.010453"/>
 			</inertial>
-            <collision>
-                <origin rpy="1.571 0 0" xyz="0 0 0" />
-                <geometry>
-                    <cylinder radius="0.06" length="0.15"/>
-                </geometry>
-            </collision>
 			<visual>
 				<origin rpy="0 0 0" xyz="0 0 0" />
@@ -196,4 +239,10 @@
 				</geometry>
 			</visual>
+            <collision>
+				<origin rpy="0 0 0" xyz="0 0 0" />
+				<geometry>
+					<mesh filename="package://dsr_description/meshes/a0509_collision/A0509_5_0.stl" scale="0.001 0.001 0.001" />
+				</geometry>
+			</collision>
             <visual>
 				<origin rpy="0 0 0" xyz="0 0 0" />
@@ -202,4 +251,10 @@
 				</geometry>
 			</visual>
+            <collision>
+				<origin rpy="0 0 0" xyz="0 0 0" />
+				<geometry>
+					<mesh filename="package://dsr_description/meshes/a0509_collision/A0509_5_1.stl" scale="0.001 0.001 0.001" />
+				</geometry>
+			</collision>
 		</link>
 		<!-- joint6 -->
@@ -226,5 +281,32 @@
 				</geometry>
 			</visual>
-		</link>
+            <collision>
+				<origin rpy="0 0 0" xyz="0 0 0" />
+				<geometry>
+					<mesh filename="package://dsr_description/meshes/a0509_collision/A0509_6_0.stl" scale="0.001 0.001 0.001" />
+				</geometry>
+			</collision>
+		</link>
+    <!-- TODO ROS base_link to Doosan Coordinates transform -->
+    <link name="${prefix}base" />
+    <joint name="${prefix}base_link-base" type="fixed">
+    <origin xyz="0 0 0" rpy="0 0 0"/>
+    <parent link="${prefix}base_link"/>
+    <child link="${prefix}base"/>
+    </joint>
+    <!-- TODO ROS-Industrial 'flange' frame: attachment point for EEF models -->
+    <link name="${prefix}flange" />
+    <joint name="${prefix}joint6-flange" type="fixed">
+    <origin xyz="0 0 0" rpy="0 0 0" />
+    <parent link="${prefix}link6" />
+    <child link="${prefix}flange" />
+    </joint>
+    <!-- TODO ROS-Industrial 'tool0' frame: all-zeros tool frame -->
+    <link name="${prefix}tool0" />
+    <joint name="${prefix}link6-tool0" type="fixed">
+      <origin xyz="0 0 0" rpy="0 0 0" />
+      <parent link="${prefix}flange" />
+      <child link="${prefix}tool0" />
+    </joint>
 		<xacro:dsr_transmission />
 		<xacro:dsr_gazebo namespace="${namespace}" />

Commit message: Use opw IK solver for a0509

File: dsr_description/xacro/macro.a0509.white.xacro (robot description, xacro)
@@ -84,5 +84,5 @@
 			<parent link="link1" />
 			<child link="link2" />
-			<origin rpy="0 -1.571 -1.571" xyz="0 0 0" />
+			<origin rpy="0 -${pi/2} -${pi/2}" xyz="0 0 0" />
 			<axis xyz="0 0 1" />
 			<limit effort="194" lower="-6.2832" upper="6.2832" velocity="3.1416"/>
@@ -137,5 +137,5 @@
 			<parent link="link2" />
 			<child link="link3" />
-			<origin rpy="0 0 1.571" xyz="0.409 0 0" />
+			<origin rpy="0 0 ${pi/2}" xyz="0.409 0 0" />
 			<axis xyz="0 0 1" />
 			<limit effort="163" lower="-2.7925" upper="2.7925" velocity="3.1416"/>
@@ -179,5 +179,5 @@
 			<parent link="link3" />
 			<child link="link4" />
-			<origin rpy="1.571 0 0" xyz="0 -0.367 0" />
+			<origin rpy="${pi/2} 0 0" xyz="0 -0.367 0" />
 			<axis xyz="0 0 1" />
 			<limit effort="50" lower="-6.2832" upper="6.2832" velocity="6.2832"/>
@@ -220,5 +220,5 @@
 			<parent link="link4" />
 			<child link="link5" />
-			<origin rpy="-1.571 0 0" xyz="0 0 0" />
+			<origin rpy="-${pi/2} 0 0" xyz="0 0 0" />
 			<axis xyz="0 0 1" />
 			<limit effort="50" lower="-6.2832" upper="6.2832" velocity="6.2832"/>
@@ -262,5 +262,5 @@
 			<parent link="link5" />
 			<child link="link6" />
-			<origin rpy="1.571 0 0" xyz="0 -0.124 0" />
+			<origin rpy="${pi/2} 0 0" xyz="0 -0.124 0" />
 			<axis xyz="0 0 1" />
 			<limit effort="50" lower="-6.2832" upper="6.2832" velocity="6.2832"/>
