Commit message: added collosion model for h2017.white (reduced *.stl)

File: dsr_description/xacro/macro.h2017.white.xacro (robot description, xacro)
@@ -4,7 +4,7 @@
 	<xacro:include filename="$(find dsr_description)/config/macro.transmission.xacro" />
 	<xacro:include filename="$(find dsr_description)/config/macro.materials.xacro" />
-	<xacro:macro name="h2017" params="namespace">
+	<xacro:macro name="h2017" params="prefix:='' namespace:=''">
 		<xacro:dsr_materials />
-		<link name="base_0">
+		<link name="base_link">
 			<inertial>
 				<mass value="8.537"/>
@@ -20,8 +20,13 @@
 				</geometry>
 			</visual>
+            <collision>
+                <geometry>
+                    <mesh filename="package://dsr_description/meshes/h2017_collision/H2017_0_0.stl" scale="0.001 0.001 0.001" />
+                </geometry>
+            </collision>
 		</link>
 		<!-- joint 1 -->
 		<joint name="joint1" type="revolute">
-			<parent link="base_0" />
+			<parent link="base_link" />
 			<child link="link1" />
 			<origin rpy="0 0 0" xyz="0 0 0.3443" />
@@ -37,9 +42,4 @@
 					izz="0.34857"/>
 			</inertial>
-            <collision>
-                <geometry>
-                    <cylinder radius="0.1" length="0.2"/>
-                </geometry>
-            </collision>
 			<visual>
 				<origin rpy="0 0 0" xyz="0 0 0" />
@@ -48,4 +48,9 @@
 				</geometry>
 			</visual>
+            <collision>
+                <geometry>
+                    <mesh filename="package://dsr_description/meshes/h2017_collision/H2017_1_0.stl" scale="0.001 0.001 0.001" />
+                </geometry>
+            </collision>
 		</link>
 		<!-- joint2 -->
@@ -53,5 +58,5 @@
 			<parent link="link1" />
 			<child link="link2" />
-			<origin rpy="0 -1.571 -1.571" xyz="0 0.0099 0" />
+			<origin rpy="0 -${pi/2} -${pi/2}" xyz="0 0.0099 0" />
 			<axis xyz="0 0 1" />
 			<limit effort="372" lower="-2.1817" upper="2.1817" velocity="1.3963"/>
@@ -65,10 +70,4 @@
 					izz="3.0015"/>
 			</inertial>
-            <collision>
-                <origin rpy="0 -1.571 0" xyz="0.3 0 0.1525" />
-                <geometry>
-                    <cylinder radius="0.08" length="0.75"/>
-                </geometry>
-            </collision>
 			<visual>
 				<origin rpy="0 0 0" xyz="0 0 0" />
@@ -77,4 +76,9 @@
 				</geometry>
 			</visual>
+            <collision>
+                <geometry>
+                    <mesh filename="package://dsr_description/meshes/h2017_collision/H2017_2_0.stl" scale="0.001 0.001 0.001" />
+                </geometry>
+            </collision>
 			<visual>
 				<origin rpy="0 0 0" xyz="0 0 0" />
@@ -83,4 +87,9 @@
 				</geometry>
 			</visual>
+            <collision>
+                <geometry>
+                    <mesh filename="package://dsr_description/meshes/h2017_collision/H2017_2_1.stl" scale="0.001 0.001 0.001" />
+                </geometry>
+            </collision>
 			<visual>
 				<origin rpy="0 0 0" xyz="0 0 0" />
@@ -89,4 +98,9 @@
 				</geometry>
 			</visual>
+            <collision>
+                <geometry>
+                    <mesh filename="package://dsr_description/meshes/h2017_collision/H2017_2_2.stl" scale="0.001 0.001 0.001" />
+                </geometry>
+            </collision>
 		</link>
 		<!-- joint3 -->
@@ -94,5 +108,5 @@
 			<parent link="link2" />
 			<child link="link3" />
-			<origin rpy="0 0 1.571" xyz="0.845 0 0" />
+			<origin rpy="0 0 ${pi/2}" xyz="0.845 0 0" />
 			<axis xyz="0 0 1" />
 			<limit effort="372" lower="-2.7925" upper="2.7925" velocity="1.7453"/>
@@ -113,4 +127,9 @@
 				</geometry>
 			</visual>
+            <collision>
+                <geometry>
+                    <mesh filename="package://dsr_description/meshes/h2017_collision/H2017_3_0.stl" scale="0.001 0.001 0.001" />
+                </geometry>
+            </collision>
 		</link>
 		<!-- joint4 -->
@@ -118,5 +137,5 @@
 			<parent link="link3" />
 			<child link="link4" />
-			<origin rpy="1.571 0 0" xyz="0 -0.734 0" />
+			<origin rpy="${pi/2} 0 0" xyz="0 -0.734 0" />
 			<axis xyz="0 0 1" />
 			<limit effort="163" lower="-6.2832" upper="6.2832" velocity="3.1416"/>
@@ -130,10 +149,4 @@
 					izz="0.078126"/>
 			</inertial>
-            <collision>
-                <origin rpy="-0.55 0 0" xyz="0 0.07 -0.3" />
-                <geometry>
-                    <cylinder radius="0.07" length="0.4"/>
-                </geometry>
-            </collision>
 			<visual>
 				<origin rpy="0 0 0" xyz="0 0 0" />
@@ -142,4 +155,9 @@
 				</geometry>
 			</visual>
+            <collision>
+                <geometry>
+                    <mesh filename="package://dsr_description/meshes/h2017_collision/H2017_4_0.stl" scale="0.001 0.001 0.001" />
+                </geometry>
+            </collision>
 			<visual>
 				<origin rpy="0 0 0" xyz="0 0 0" />
@@ -148,4 +166,9 @@
 				</geometry>
 			</visual>
+            <collision>
+                <geometry>
+                    <mesh filename="package://dsr_description/meshes/h2017_collision/H2017_4_1.stl" scale="0.001 0.001 0.001" />
+                </geometry>
+            </collision>
 		</link>
 		<!-- joint5 -->
@@ -153,5 +176,5 @@
 			<parent link="link4" />
 			<child link="link5" />
-			<origin rpy="-1.571 0 0" xyz="0 0 0" />
+			<origin rpy="-${pi/2} 0 0" xyz="0 0 0" />
 			<axis xyz="0 0 1" />
 			<limit effort="96" lower="-6.2832" upper="6.2832" velocity="3.1416"/>
@@ -166,10 +189,4 @@
 					izz="0.014587"/>
 			</inertial>
-            <collision>
-                <origin rpy="1.571 0 0" xyz="0 0 0" />
-                <geometry>
-                    <cylinder radius="0.08" length="0.15"/>
-                </geometry>
-            </collision>
 			<visual>
 				<origin rpy="0 0 0" xyz="0 0 0" />
@@ -178,4 +195,9 @@
 				</geometry>
 			</visual>
+            <collision>
+                <geometry>
+                    <mesh filename="package://dsr_description/meshes/h2017_collision/H2017_5_0.stl" scale="0.001 0.001 0.001" />
+                </geometry>
+            </collision>
 		</link>
 		<!-- joint6 -->
@@ -183,5 +205,5 @@
 			<parent link="link5" />
 			<child link="link6" />
-			<origin rpy="1.571 0 0" xyz="0 -0.121 0" />
+			<origin rpy="${pi/2} 0 0" xyz="0 -0.121 0" />
 			<axis xyz="0 0 1" />
 			<limit effort="50" lower="-6.2832" upper="6.2832" velocity="3.927"/>
@@ -202,5 +224,31 @@
 				</geometry>
 			</visual>
-		</link>
+            <collision>
+                <geometry>
+                    <mesh filename="package://dsr_description/meshes/h2017_collision/H2017_6_0.stl" scale="0.001 0.001 0.001" />
+                </geometry>
+            </collision>
+		</link>
+    <!-- TODO ROS base_link to Doosan Coordinates transform -->
+    <link name="${prefix}base" />
+    <joint name="${prefix}base_link-base" type="fixed">
+    <origin xyz="0 0 0" rpy="0 0 0"/>
+    <parent link="${prefix}base_link"/>
+    <child link="${prefix}base"/>
+    </joint>
+    <!-- TODO ROS-Industrial 'flange' frame: attachment point for EEF models -->
+    <link name="${prefix}flange" />
+    <joint name="${prefix}joint6-flange" type="fixed">
+    <origin xyz="0 0 0" rpy="0 0 0" />
+    <parent link="${prefix}link6" />
+    <child link="${prefix}flange" />
+    </joint>
+    <!-- TODO ROS-Industrial 'tool0' frame: all-zeros tool frame -->
+    <link name="${prefix}tool0" />
+    <joint name="${prefix}link6-tool0" type="fixed">
+      <origin xyz="0 0 0" rpy="0 0 0" />
+      <parent link="${prefix}flange" />
+      <child link="${prefix}tool0" />
+    </joint>
 		<xacro:dsr_transmission />
 		<xacro:dsr_gazebo namespace="${namespace}" />
